File: sensormodule.kicad_pcb (KiCad board)
At the start: 2 copper layers, 20 x 15 mm, 17 parts, among them X1 [Crystal]_32.768KHz

Commit message: 1
Parts:
- added C12: 16pF, Kylian:[0402] Capacitor, F.Cu at (87.8, 85.0)
- added C13: 16pF, Kylian:[0402] Capacitor, F.Cu at (89.8, 85.0)
- added R3: 1M, Kylian:[0402] Resistor, F.Cu at (87.8, 86.0)
- added X2: 16MHz, Kylian:[XTAL] 2mmx1.6mm, F.Cu at (89.0, 90.6)
- X1: value [Crystal]_32.768KHz -> 32.768KHz
- moved C11 16.4 mm to (87.8, 87.0), turned to 180 degrees
- moved C10 12.7 mm to (89.8, 86.0), turned to 180 degrees
- moved C6 11.3 mm to (88.8, 78.6)
- moved X1 10.7 mm to (89.0, 88.4), turned to 180 degrees
- moved R2 3.83 mm to (89.8, 84.0)
- moved C5 3.79 mm to (87.8, 84.0)
- moved R1 2.90 mm to (89.8, 83.0)
- moved C4 2.84 mm to (87.8, 83.0)
- moved C8 2.83 mm to (87.8, 81.0)
- moved C1 2.50 mm to (89.8, 81.0)
- moved U1 2.24 mm to (93.8, 85.4)
- moved U2 2.24 mm to (93.8, 80.4)
- moved C9 1.99 mm to (89.8, 82.0)
- moved C2 1.94 mm to (87.8, 80.0)
- moved C3 1.90 mm to (87.8, 82.0)
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Connections:
- U2 pad 10: unconnected-(U2-XC1-Pad10) -> Net-(U2-XC1)
- U2 pad 9: unconnected-(U2-XC2-Pad9) -> Net-(U2-XC2)

Commit message: update
Parts:
- added C14: 4.7pF, Kylian:[0402] Capacitor, F.Cu at (103.5, 79.4)
- added C15: 2.2nF, Kylian:[0402] Capacitor, F.Cu at (103.5, 80.4)
- added C16: 1.5pF, Kylian:[0402] Capacitor, F.Cu at (103.5, 81.4)
- added C17: 1pF, Kylian:[0402] Capacitor, F.Cu at (103.5, 82.4)
- added J1: [Header]_4-Pos_1.27mm, Kylian:[Header] 1.27mm 4-Position, F.Cu at (89.6, 80.2)
- added L1: 8.2nH, Kylian:[0402] Inductor, F.Cu at (103.5, 83.4)
- added L2: 3.9nH, Kylian:[0402] Inductor, F.Cu at (103.5, 84.4)
- added L3: 2.7nH, Kylian:[0402] Inductor, F.Cu at (103.5, 85.4)
- moved C13 10.3 mm to (98.7, 90.3), turned to 90 degrees
- moved S1 10.3 mm to (95.7, 79.2)
- moved C8 10.2 mm to (94.7, 88.6)
- moved C1 9.35 mm to (99.1, 80.0), turned to -90 degrees
- moved R3 9.34 mm to (96.8, 88.6), turned to 180 degrees
- moved R2 9.27 mm to (98.9, 82.1), turned to 180 degrees
- moved C2 9.09 mm to (91.5, 88.3), turned to 180 degrees
- moved C12 8.84 mm to (94.9, 90.3), turned to 90 degrees
- moved X2 7.78 mm to (96.8, 90.3), turned to 180 degrees
- moved C7 7.28 mm to (96.8, 82.1), turned to 180 degrees
- moved C5 7.04 mm to (92.2, 89.5), turned to 180 degrees
- moved U2 5.49 mm to (96.1, 85.4)
- moved C4 5.30 mm to (87.6, 88.3)
- moved C9 4.88 mm to (94.7, 82.1)
- moved U1 4.33 mm to (89.5, 85.4), turned to 90 degrees
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Connections:
- net Net-(U1-BOOT0) renamed /BOOT0
- net Net-(U1-NRST) renamed /NRST
- net Net-(U1-PC14-OSC32_IN) renamed /OSC32_IN
- net Net-(U1-PC15-OSC32_OUT) renamed /OSC32_OUT
- net Net-(U2-DVDD) renamed /DVDD
- net Net-(U2-IREF) renamed /IREF
- net Net-(U2-XC1) renamed /OSC16_2
- net Net-(U2-XC2) renamed /OSC16_1
- C7 pad 2: Net-(C7-Pad2) -> +BATT
- C8 pad 2: Net-(C7-Pad2) -> +BATT
- U1 pad 10: /CS -> unconnected-(U1-PA4-Pad10)
- U1 pad 12: /MISO -> unconnected-(U1-PA6-Pad12)
- U1 pad 14: unconnected-(U1-PB0-Pad14) -> /MISO
- U1 pad 15: unconnected-(U1-PB1-Pad15) -> /CS
- U1 pad 18: unconnected-(U1-PA8-Pad18) -> /CE
- U1 pad 9: /CE -> unconnected-(U1-PA3-Pad9)
- U2 pad 11: unconnected-(U2-VDD_PA-Pad11) -> Net-(U2-VDD_PA)
- U2 pad 12: unconnected-(U2-ANT1-Pad12) -> Net-(U2-ANT1)
- U2 pad 13: unconnected-(U2-ANT2-Pad13) -> Net-(U2-ANT2)
- U2 pad 15: Net-(C7-Pad2) -> +BATT
- U2 pad 18: Net-(C7-Pad2) -> +BATT
- U2 pad 7: Net-(C7-Pad2) -> +BATT
Routing:
- net +BATT: track 0.00 -> 37.0 mm, vias 0 -> 3
- net /NRST: track 0.00 -> 16.2 mm, vias 0 -> 2
- net /SWDIO: track 0.00 -> 5.80 mm
- net /OSC16_2: track 0.00 -> 5.51 mm
- net /CE: track 0.00 -> 5.26 mm, vias 0 -> 2
- net /SWCLK: track 0.00 -> 5.14 mm
- net /MOSI: track 0.00 -> 4.25 mm
- net /OSC16_1: track 0.00 -> 4.17 mm
- net /OSC32_IN: track 0.00 -> 4.16 mm
- net /MISO: track 0.00 -> 4.05 mm
- net /SCK: track 0.00 -> 3.92 mm, vias 0 -> 2
- net /OSC32_OUT: track 0.00 -> 3.81 mm
- net /CS: track 0.00 -> 3.77 mm
- net /IRQ: track 0.00 -> 3.66 mm
- net /IREF: track 0.00 -> 1.84 mm
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- added copper zone on B.Cu, net GND
- added copper zone on F.Cu, net GND
- added copper zone on In1.Cu, net GND
- added copper zone on In2.Cu, net GND
Other:
- copper layers 2 -> 4
